File: Bus-tester.kicad_pcb (KiCad board)
At the start: 2 copper layers, 110 x 60 mm, 79 parts, among them J1 POWER, J10 In_Reg, J11 Out_Reg, J12 POWER, J2 POWER, J3 C1_out, J4 C2_out, J5 C3_out, J6 C4_out, J7 Out_sw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

Commit message: make PCB marking parameterized
Other:
- board text added: "${TITLE} ${REVISION}"
- board text removed: "Bus tester v1.0"
Changed lines of the file:
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@@
   )
   (paper "A4")
+  (title_block
+    (title "Bus tester")
+    (rev "v1.0")
+  )
   (layers
     (0 "F.Cu" signal)
@@
     (effects (font (size 1 1) (thickness 0.15)))
   )
-  (gr_text "Bus tester\nv1.0" (at 34.29 57.785) (layer "F.SilkS")
+  (gr_text "${TITLE}\n${REVISION}" (at 34.29 57.785) (layer "F.SilkS")
     (effects (font (size 3 3) (thickness 0.4)))
   )
