File: Bus-tester.kicad_pcb (KiCad board)
At the start: 2 copper layers, 110 x 60 mm, 79 parts, among them J1 POWER, J10 In_Reg, J11 Out_Reg, J12 POWER, J2 POWER, J3 C1_out, J4 C2_out, J5 C3_out, J6 C4_out, J7 Out_sw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

Commit message: change resistor arrays footprints
Parts:
- RN1, RN10, RN11, RN2, RN4, RN5, RN6, RN7, RN8, RN9: footprint Resistor_SMD:R_Array_Convex_4x1206 -> Resistor_SMD:R_Array_Convex_4x0603
Routing:
- net VCC: track 321.5 -> 309.7 mm
- net Net-(RN1D-R4.2): track 14.2 -> 15.8 mm
- net Net-(D21-K): track 4.20 -> 5.70 mm
- net Net-(D14-K): track 4.20 -> 5.70 mm
- net Net-(D9-K): track 4.20 -> 5.70 mm
- net Net-(D6-K): track 4.20 -> 5.70 mm
- net Net-(D18-K): track 4.20 -> 5.70 mm
- net Net-(D17-K): track 4.20 -> 5.70 mm
- net Net-(D13-K): track 4.20 -> 5.70 mm
- net Net-(D10-K): track 4.20 -> 5.70 mm
- net Net-(D26-A): track 15.3 -> 16.4 mm
- net Net-(D25-A): track 15.3 -> 16.4 mm
- net /~{D_{7}}: track 44.6 -> 45.5 mm
- net /~{D_{0}}: track 44.4 -> 45.4 mm
- net Net-(RN1A-R1.2): track 53.2 -> 54.1 mm
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